Commit message: Update
New links and joints as reference for path

File: URDF Codes/articulatedRobot.urdf (robot description, URDF)
Before this commit: robot articulated_robot, 12 links, 11 joints
Links:
- added link workstation
Joints:
- added joint transformation: type fixed, parent base_link, child workstation, origin xyz=0 0 0 rpy=0 0 0

File: URDF Codes/articulatedRobot2.urdf (robot description, URDF)
Before this commit: robot articulated_robot, 14 links, 13 joints
Links:
- added link workstation
Joints:
- added joint transformation: type fixed, parent base_link, child workstation, origin xyz=0 0 0 rpy=0 0 0

File: URDF Codes/gantryRobot.urdf (robot description, URDF)
Before this commit: robot gantry_robot, 5 links, 4 joints
Links:
- added link workstation
Joints:
- added joint transformation: type fixed, parent base_link, child workstation, origin xyz=0 0 0 rpy=0 0 0

File: URDF Codes/scaraRobot.urdf (robot description, URDF)
Before this commit: robot scara_robot, 6 links, 5 joints
Links:
- added link workstation
Joints:
- removed joint prismatic1_z
- removed joint prismatic2_x
- removed joint prismatic3_x
- added joint design_prismatic1_z: type prismatic, parent base_link, child virtual_link1_z, origin xyz=0 0 0.1 rpy=0 0 0, axis 0 0 1, limit lower=0 upper=10 effort=1000 velocity=0.5
- added joint design_prismatic2_x: type prismatic, parent link1, child virtual_link2_x, origin xyz=0 0 0 rpy=0 0 0, axis 1 0 0, limit lower=0 upper=4 effort=500 velocity=0.2
- added joint design_prismatic3_x: type prismatic, parent link2, child end_effector, origin xyz=0 0 0 rpy=0 0 0, axis 1 0 0, limit lower=0 upper=4 effort=500 velocity=0.2
- added joint transformation: type fixed, parent base_link, child workstation, origin xyz=0 0 0 rpy=0 0 0
