Commit message: Update
This file is for testing the optimization and simulation envoronment

File: URDF Codes/scaraRobot.urdf (robot description, URDF)
Before this commit: robot scara_robot, 7 links, 6 joints
Joints:
- joint design_prismatic1_z: origin xyz=0 0 0.1 rpy=0 0 0 -> xyz=0 0 0.0 rpy=0 0 0
- joint rotative1: limit lower=-6.28 upper=6.28 effort=1000 velocity=0.5 -> lower=-6.28 upper=6.28 effort=1000 velocity=1
- joint rotative2: limit lower=-6.28 upper=6.28 effort=1000 velocity=0.5 -> lower=-6.28 upper=6.28 effort=1000 velocity=1
